File: examples/ESP-DMX/ESP-DMX.brd (EAGLE design)
At the start: 41.6 x 71.1 mm, 12 parts, among them IC1 MAX481CPA

Commit message: Change input pullup resistor
Parts:
- moved R1 17.3 mm to (25.4, 31.8), turned to 90 degrees
Connections:
- new net N$7: HUZZAH-TX.8, R1.2
- net N$8: now also R1.1; no longer R1.2
- net VCC: no longer R1.1
Routing:
- net N$8: track 34.9 -> 49.5 mm
- net VCC: track 75.0 -> 66.8 mm
- net N$7: track 0.00 -> 6.35 mm
Changed lines of the file:
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@@
 <?xml version="1.0" encoding="utf-8"?>
 <!DOCTYPE eagle SYSTEM "eagle.dtd">
-<eagle version="7.5.0">
+<eagle version="7.7.0">
 <drawing>
 <settings>
@@
 <attribute name="VALUE" x="21.59" y="5.715" size="1.27" layer="27"/>
 </element>
-<element name="R1" library="RBBB" package="RESISTOR" value="10k" x="20.32" y="15.24" rot="R180"/>
+<element name="R1" library="RBBB" package="RESISTOR" value="10k" x="25.4" y="31.75" rot="R90"/>
 <element name="U$3" library="holes" package="2,8" value="" x="5.08" y="67.31"/>
 <element name="U$4" library="holes" package="2,8" value="" x="36.83" y="67.31"/>
@@
 <contactref element="IC1" pad="8"/>
 <contactref element="PWR/SW" pad="2"/>
-<contactref element="R1" pad="1"/>
 <wire x1="11.43" y1="55.499" x2="11.43" y2="55.88" width="0.254" layer="16"/>
 <wire x1="3.8862" y1="55.4228" x2="11.43" y2="55.499" width="0.254" layer="16"/>
@@
 <wire x1="25.3492" y1="24.1554" x2="3.7592" y2="30.5054" width="0.254" layer="16"/>
 <wire x1="25.3492" y1="24.1554" x2="25.4" y2="20.32" width="0.254" layer="16"/>
-<wire x1="25.4" y1="20.32" x2="22.86" y2="15.24" width="0.4064" layer="16"/>
 <contactref element="(C1)" pad="2"/>
 <wire x1="25.4" y1="11.43" x2="24.13" y2="11.43" width="0.4064" layer="16"/>
 <wire x1="25.4" y1="8.89" x2="25.4" y2="11.43" width="0.4064" layer="16"/>
 <wire x1="25.4" y1="11.43" x2="25.4" y2="15.24" width="0.4064" layer="16"/>
-<wire x1="25.4" y1="15.24" x2="22.86" y2="15.24" width="0.4064" layer="16"/>
+<wire x1="25.4" y1="15.24" x2="25.4" y2="20.32" width="0" layer="19" extent="16-16"/>
 </signal>
 <signal name="N$2">
@@
 <signal name="N$8">
 <contactref element="PWR/SW" pad="4"/>
+<wire x1="33.02" y1="29.21" x2="33.02" y2="8.89" width="0.4064" layer="1"/>
+<wire x1="33.02" y1="8.89" x2="30.48" y2="8.89" width="0.4064" layer="1"/>
 <contactref element="HUZZAH" pad="4"/>
-<contactref element="R1" pad="2"/>
-<wire x1="17.78" y1="15.24" x2="15.24" y2="20.32" width="0.4064" layer="16"/>
-<wire x1="30.48" y1="8.89" x2="30.48" y2="3.81" width="0.4064" layer="16"/>
-<wire x1="30.48" y1="3.81" x2="17.78" y2="3.81" width="0.4064" layer="16"/>
-<wire x1="17.78" y1="3.81" x2="17.78" y2="15.24" width="0.4064" layer="16"/>
+<contactref element="R1" pad="1"/>
+<wire x1="33.02" y1="29.21" x2="25.4" y2="29.21" width="0.4064" layer="1"/>
+<wire x1="25.4" y1="29.21" x2="15.24" y2="29.21" width="0.4064" layer="1"/>
+<wire x1="15.24" y1="29.21" x2="15.24" y2="20.32" width="0.4064" layer="1"/>
 </signal>
 <signal name="N$1">
@@
 <wire x1="11.43" y1="64.77" x2="11.43" y2="67.31" width="0.4064" layer="16"/>
 </signal>
+<signal name="N$7">
+<contactref element="HUZZAH-TX" pad="8"/>
+<contactref element="R1" pad="2"/>
+<wire x1="25.4" y1="40.64" x2="25.4" y2="34.29" width="0.4064" layer="16"/>
+</signal>
 </signals>

Commit message: add rdm support
Parts:
- added R3: 10Kohm, RBBB:RESISTOR
Connections:
- net GND: now also R3.1
- net N$5: now also R3.2
Routing:
- net GND: track 87.0 -> 98.4 mm
- net N$5: track 7.92 -> 16.8 mm
Changed lines of the file:
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@@
 <attribute name="VALUE" x="13.081" y="11.176" size="1.27" layer="27" ratio="10"/>
 </element>
+<element name="R3" library="RBBB" package="RESISTOR" value="10Kohm" x="12.7" y="31.75" rot="R180"/>
 </elements>
 <signals>
@@
 <wire x1="19.05" y1="55.88" x2="19.05" y2="60.96" width="0.4064" layer="16"/>
 <contactref element="HUZZAH-TX" pad="10"/>
-<wire x1="30.48" y1="20.32" x2="30.48" y2="40.64" width="0.4064" layer="16"/>
+<wire x1="30.48" y1="20.32" x2="30.48" y2="31.75" width="0.4064" layer="16"/>
+<wire x1="30.48" y1="31.75" x2="30.48" y2="40.64" width="0.4064" layer="16"/>
 <wire x1="30.48" y1="40.64" x2="30.48" y2="44.45" width="0.4064" layer="16"/>
 <wire x1="30.48" y1="44.45" x2="25.4" y2="44.45" width="0.4064" layer="16"/>
@@
 <wire x1="30.48" y1="13.97" x2="30.48" y2="20.32" width="0.4064" layer="16"/>
 <contactref element="(C1)" pad="1"/>
-<wire x1="22.86" y1="6.35" x2="19.05" y2="6.35" width="0.4064" layer="16"/>
 <wire x1="19.05" y1="6.35" x2="19.05" y2="11.43" width="0.4064" layer="16"/>
 <wire x1="22.86" y1="6.35" x2="19.05" y2="6.35" width="0.4064" layer="16"/>
+<contactref element="R3" pad="1"/>
+<wire x1="15.24" y1="31.75" x2="30.48" y2="31.75" width="0.4064" layer="16"/>
 </signal>
 <signal name="VCC">
@@
 <wire x1="10.16" y1="44.45" x2="11.43" y2="46.99" width="0.4064" layer="16" curve="-90"/>
 <wire x1="11.43" y1="46.99" x2="11.43" y2="48.26" width="0.4064" layer="16"/>
+<contactref element="R3" pad="2"/>
+<wire x1="10.16" y1="31.75" x2="10.16" y2="40.64" width="0.4064" layer="16"/>
 </signal>
 <signal name="N$8">
